Commit message: end-effector offset to null in jacobian

File: sawyer_description/urdf/sawyer_base.urdf.xacro (robot description, xacro)
@@ -430,5 +430,5 @@
   </link>
   <joint name="right_hand" type="fixed">
-    <origin rpy="0 0 1.570796" xyz="0 0 0.0245"/>
+    <origin rpy="0 0 1.570796" xyz="0.001 0.001 0.100"/>
     <axis xyz="0 0 1"/>
     <parent link="right_l6"/>
